File: Digital.sch (KiCad schematic (older format))
At the start: 49 parts, among them J1 Conn_02x05_Odd_Even_MountingP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, Q1 Q_NMOS_GSD, U1 STM32F746VGTx, U2 MOUDLE-BLUETOOTH-HC-05(34P-27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, Y1 25MHz, Y2 32kHz

Commit message: Footprint changed in Y1
Parts:
- U2: symbol myKicadlib:MOUDLE-BLUETOOTH-HC-05(34P-27X13MM) -> Digital-rescue:MOUDLE-BLUETOOTH-HC-05(34P-27X13MM)-myKicadlib
- Y1: footprint Crystals:Crystal_SMD_2520-4pin_2.5x2.0mm -> User_library:OSCCC320X250X60N
Changed lines of the file:
@@
 F 0 "Y1" V 2300 3150 50  0000 L CNN
 F 1 "25MHz" V 2300 2850 50  0000 L CNN
-F 2 "Crystals:Crystal_SMD_2520-4pin_2.5x2.0mm" H 2300 3200 50  0001 C CNN
+F 2 "User_library:OSCCC320X250X60N" H 2300 3200 50  0001 C CNN
 F 3 "https://es.rs-online.com/web/p/osciladores-crystal/1732365/" H 2300 3200 50  0001 C CNN
 	1    2300 3200
@@
 	2700 6050 2400 6050
 $Comp
-L myKicadlib:MOUDLE-BLUETOOTH-HC-05(34P-27X13MM) U2
+L Digital-rescue:MOUDLE-BLUETOOTH-HC-05(34P-27X13MM)-myKicadlib U2
 U 1 1 5BCE726A
 P 8150 2100
